File: kicad/Pixel_Star.kicad_pcb (KiCad board)
At the start: 2 copper layers, 95.3 x 91.1 mm, 55 parts, among them J1 USB_C_Female, J2 Conn_01x04_Female, SW1 SW_Push, SW2 SW_Push, SW3 SW_Push, U1 AMS1117-3.3, U2 STM32G030F6P6TR, U3 SN74LV1T34DBVR

Commit message: Improve PCB labels - SWD connector, Reset button
Other:
- board text added: "3.3V"
- board text added: "CLK"
- board text added: "DIO"
- board text added: "GND"
- board text added: "RST"
- board text added: "SWD"
Changed lines of the file:
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@@
     (property "Sheetname" "")
     (attr smd)
-    (fp_text reference "J2" (at 0 -4.4 172) (layer "F.SilkS")
+    (fp_text reference "J2" (at 6.87234 -2.585198 262) (layer "F.SilkS")
       (effects (font (size 1 1) (thickness 0.15)))
     )
@@
     (property "Sheetname" "")
     (attr smd)
-    (fp_text reference "SW3" (at 0 -2.6 90) (layer "F.SilkS")
+    (fp_text reference "SW3" (at 0 -2.6 90) (layer "F.Fab")
       (effects (font (size 1 1) (thickness 0.15)))
     )
@@
     (effects (font (size 1.5 1.5) (thickness 0.3)))
   )
+  (gr_text "SWD" (at 167.64 80.721934 262) (layer "F.SilkS")
+    (effects (font (size 1 1) (thickness 0.15)))
+  )
   (gr_text "V1.0" (at 114.3254 111.5822 -45) (layer "F.SilkS")
     (effects (font (size 1.5 1.5) (thickness 0.3)))
   )
+  (gr_text "GND" (at 157.960469 83.857103 82) (layer "F.SilkS")
+    (effects (font (size 1 1) (thickness 0.15)))
+  )
+  (gr_text "RST" (at 135.500275 67.473875 90) (layer "F.SilkS")
+    (effects (font (size 1 1) (thickness 0.15)))
+  )
+  (gr_text "CLK" (at 159.334924 84.02891 82) (layer "F.SilkS")
+    (effects (font (size 1 1) (thickness 0.15)))
+  )
+  (gr_text "DIO" (at 160.6712 84.219806 82) (layer "F.SilkS")
+    (effects (font (size 1 1) (thickness 0.15)))
+  )
+  (gr_text "3.3V" (at 162.007475 84.773406 82) (layer "F.SilkS")
+    (effects (font (size 1 1) (thickness 0.15)))
+  )
   (segment (start 140.2966 119.7486) (end 140.9192 119.126) (width 0.5) (layer "F.Cu") (net 1))
